Commit message: computed proper velocity limits for LSS servos

File: urdf/lss.xacro (robot description, xacro)
@@ -5,5 +5,5 @@
     <xacro:property name="ht1_max_torque_static" value="6.8439285" />
     <xacro:property name="ht1_max_torque_dynamic" value="6.5687857" />
-    <xacro:property name="ht1_max_velocity" value="0.58" />
+    <xacro:property name="ht1_max_velocity" value="6.283" />
     <!--
           todo: need to update these values to real ones
@@ -12,9 +12,9 @@
     <xacro:property name="st1_max_torque_static" value="6.8439285" />
     <xacro:property name="st1_max_torque_dynamic" value="6.5687857" />
-    <xacro:property name="st1_max_velocity" value="0.58" />
+    <xacro:property name="st1_max_velocity" value="6.283" />
     <!-- torques in N-m, velocity in rads/sec for no-load -->
     <xacro:property name="hs1_max_torque_static" value="6.8439285" />
     <xacro:property name="hs1_max_torque_dynamic" value="6.5687857" />
-    <xacro:property name="hs1_max_velocity" value="0.58" />
+    <xacro:property name="hs1_max_velocity" value="10.47" />
     <xacro:macro name="limits-HT1" params="lower_limit=-3.14 upper_limit=3.14">
         <limit

Commit message: updated ST1 torque values and Inertials. Fixed issue preventing joints from moving (due to spring settings)

File: urdf/lss.xacro (robot description, xacro)
@@ -10,6 +10,6 @@
     -->
     <!-- torques in N-m, velocity in rads/sec for no-load -->
-    <xacro:property name="st1_max_torque_static" value="6.8439285" />
-    <xacro:property name="st1_max_torque_dynamic" value="6.5687857" />
+    <xacro:property name="st1_max_torque_static" value="1.372931" />
+    <xacro:property name="st1_max_torque_dynamic" value="0.2745862" />
     <xacro:property name="st1_max_velocity" value="6.283" />
     <!-- torques in N-m, velocity in rads/sec for no-load -->
@@ -39,11 +39,11 @@
                 velocity="${st1_max_velocity}" />
         <safety_controller
-                k_position="0.3"
+                k_position="10"
                 k_velocity="100"
-                soft_lower_limit="-3.1"
-                soft_upper_limit="3.1" />
+                soft_lower_limit="-3.14"
+                soft_upper_limit="3.14" />
         <dynamics
-                damping="0.01"
-                friction="9E-05" />
+                damping="0.0"
+                friction="0.0" />
     </xacro:macro>
     <xacro:macro name="limits-HS1" params="lower_limit=-3.14 upper_limit=3.14">
@@ -109,4 +109,7 @@
     </xacro:macro>
     <xacro:macro name="gzjoint" params="ref preserve:=0">
+      <!-- no gz joint parameters for now -->
+    </xacro:macro>
+    <xacro:macro name="gzjoint-springy" params="ref preserve:=0">
         <gazebo reference="${ref}">
             <xacro:if value="${preserve}">
@@ -114,6 +117,15 @@
             </xacro:if>
             <implicitSpringDamper>true</implicitSpringDamper>
-            <springStiffness>100</springStiffness>
-            <springReference>0.01</springReference>
+            <!--
+               Spring stiffness coefficient
+               The stiffness coefficient causes a torque (force for prismatic
+               joints) to be applied based on the current joint position.
+               At the spring_reference position no torque is applied.
+               At any other position a torque is applied to the joint with a
+               direction towards the spring_reference position.
+               torque = spring_stiffness * (spring_reference - current_position)
+            -->
+            <springStiffness>0.15</springStiffness>
+            <springReference>0.5</springReference>
             <!-- untuned parameters -->
             <!--stopCfm>0.2</stopCfm>
@@ -203,15 +215,15 @@
             <inertial>
                 <origin
-                        xyz="0 0 0"
+                        xyz="-0.0187 0.0111 -0.000095622"
                         rpy="0 0 0" />
                 <mass
-                        value="0.355132365146695" />
+                        value="0.08678" />
                 <inertia
-                        ixx="0"
-                        ixy="0"
-                        ixz="0"
-                        iyy="0"
-                        iyz="0"
-                        izz="0" />
+                        ixx="0.000032833"
+                        ixy="-0.000018518"
+                        ixz="0.000000085540"
+                        iyy="0.000049952"
+                        iyz="-0.000000088136"
+                        izz="0.000074803" />
             </inertial>
             <visual>

Commit message: moved meshes and configured automatic model paths via env-hooks

File: urdf/lss.xacro (robot description, xacro)
@@ -239,5 +239,5 @@
                 </xacro:if>
                 <geometry>
-                    <mesh filename="package://lss_hexapod/meshes/LSS-Servo-Aluminum.dae" />
+                    <mesh filename="model://lss_humanoid/LSS-Servo-Aluminum.dae" />
                 </geometry>
                 <material name="white" />
@@ -248,5 +248,5 @@
                         rpy="0 0 0" />
                 <geometry>
-                    <mesh filename="package://lss_hexapod/meshes/LSS-Servo-Aluminum.dae" />
+                    <mesh filename="model://lss_humanoid/LSS-Servo-Aluminum.dae" />
                 </geometry>
             </collision>

File: urdf/lss_humanoid.xacro.urdf (robot description, URDF)
Before this commit: robot lss_humanoid, 23 links, 4 joints
Links:
- link Backpack: geometry collision mesh filename=model://lss_humanoid/collision/Backpack.STL; visual mesh filename=model://lss_humanoid/Backpack.dae
- link LFootPitch: geometry collision mesh filename=model://lss_humanoid/collision/LFootPitch.STL; visual mesh filename=model://lss_humanoid/LFootPitch.dae
- link LFootRoll: geometry collision mesh filename=model://lss_humanoid/collision/LFootRoll.STL; visual mesh filename=model://lss_humanoid/LFootRoll.STL
- link LHipPitch: geometry collision mesh filename=model://lss_humanoid/collision/LHipPitch.STL; visual mesh filename=model://lss_humanoid/LHipPitch.dae
- link LHipRoll: geometry collision mesh filename=model://lss_humanoid/collision/LHipRoll.STL; visual mesh filename=model://lss_humanoid/LHipRoll.dae
- link LHipYaw: geometry collision mesh filename=model://lss_humanoid/collision/LHipYaw.STL; visual mesh filename=model://lss_humanoid/LHipYaw.STL
- link LHumerus: geometry collision mesh filename=model://lss_humanoid/collision/LHumerus.STL; visual mesh filename=model://lss_humanoid/LHumerus.dae
- link LKnee: geometry collision mesh filename=model://lss_humanoid/collision/LKnee.STL; visual mesh filename=model://lss_humanoid/LKnee.STL
- link LRadius: geometry collision mesh filename=model://lss_humanoid/collision/LRadius.STL; visual mesh filename=model://lss_humanoid/LRadius.STL
- link LShoulder: geometry collision mesh filename=model://lss_humanoid/collision/LShoulder.STL; visual mesh filename=model://lss_humanoid/LShoulder.STL
- link RFootPitch: geometry collision mesh filename=model://lss_humanoid/collision/LFootPitch.STL; visual mesh filename=model://lss_humanoid/LFootPitch.dae
- link RFootRoll: geometry collision mesh filename=model://lss_humanoid/collision/LFootRoll.STL; visual mesh filename=model://lss_humanoid/LFootRoll.STL
- link RHipPitch: geometry collision mesh filename=model://lss_humanoid/collision/LHipPitch.STL; visual mesh filename=model://lss_humanoid/LHipPitch.dae
- link RHipRoll: geometry collision mesh filename=model://lss_humanoid/collision/LHipRoll.STL; visual mesh filename=model://lss_humanoid/LHipRoll.dae
- link RHipYaw: geometry collision mesh filename=model://lss_humanoid/collision/LHipYaw.STL; visual mesh filename=model://lss_humanoid/LHipYaw.STL
- link RHumerus: geometry collision mesh filename=model://lss_humanoid/collision/LHumerus.STL; visual mesh filename=model://lss_humanoid/LHumerus.dae
- link RKnee: geometry collision mesh filename=model://lss_humanoid/collision/LKnee.STL; visual mesh filename=model://lss_humanoid/LKnee.STL
- link RRadius: geometry collision mesh filename=model://lss_humanoid/collision/LRadius.STL; visual mesh filename=model://lss_humanoid/LRadius.STL
- link RShoulder: geometry collision mesh filename=model://lss_humanoid/collision/LShoulder.STL; visual mesh filename=model://lss_humanoid/LShoulder.STL
- link base_link: geometry collision mesh filename=model://lss_humanoid/collision/Torso.STL; visual mesh filename=model://lss_humanoid/Torso.dae
- link l_sole: geometry collision box size=0.120 0.064 0.002; visual mesh filename=model://lss_humanoid/LSole.STL
- link r_sole: geometry collision box size=0.120 0.064 0.002; visual mesh filename=model://lss_humanoid/LSole.STL

Commit message: added ign sim parameter

File: urdf/lss.xacro (robot description, xacro)
@@ -1,4 +1,6 @@
 <?xml version="1.0" encoding="utf-8"?>
 <lss xmlns:xacro="http://www.ros.org/wiki/xacro">
+    <xacro:arg name="sim" default="ign" />
+    <xacro:property name="sim" value="arg ign" />
     <xacro:property name="ros2_controls" value="true" />
     <!-- torques in N-m, velocity in rads/sec for no-load -->

Commit message: added low poly mesh for ST1 servo

File: urdf/lss.xacro (robot description, xacro)
@@ -245,10 +245,19 @@
                 <material name="white" />
             </visual>
-            <collision>
-                <origin
-                        xyz="0 0 0"
-                        rpy="0 0 0" />
-                <geometry>
-                    <mesh filename="model://lss_humanoid/LSS-Servo-Aluminum.dae" />
+	    <collision>
+                <xacro:if value="${not reverse}">
+                    <origin
+                        xyz="${-0.01915} 0.0125 0"
+                        rpy="0 ${mirror_rot} 0" />
+                </xacro:if>
+                <xacro:if value="${reverse}">
+                    <origin
+                            xyz="${-0.01915} 0.0125 0"
+                            rpy="3.14159 ${mirror_rot} 0" />
+                </xacro:if>
+		<geometry>
+			<!--box size="0.0383 0.051 0.025"/-->
+			<mesh filename="model://lss_humanoid/collision/LSS-Servo-Aluminum.stl" />
+			<!--mesh filename="model://lss_humanoid/LSS-Servo-Aluminum.dae" /-->
                 </geometry>
             </collision>
